File: PCB/pico.kicad_pcb (KiCad board)
At the start: 2 copper layers, 40 x 75 mm, 14 parts, among them J1 Barrel_Jack_MountingPin, J2 Conn_01x03, J3 Conn_01x04, J4 Conn_01x02_Pin, U1 MPU-6050

Commit message: Add Version !.0
Routing:
- added copper zone on B.Cu, net GNDREF
- added copper zone on F.Cu, net GNDREF
Other:
- board text added: "3.3VDC Out"
- board text added: "5VDC Out"
- board text added: "Din"
- board text added: "GND"
- board text added: "Internship Technical Test Assignment"
- board text added: "SCL"
- board text added: "SDA"
- board text added: "V 1.0"
- board text added: "Yens & Yens"
Changed lines of the file:
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@@
 		(tags "connector JST PH horizontal")
 		(property "Reference" "J2"
-			(at 2 -2.55 0)
+			(at -3.5 2.5 0)
 			(layer "F.SilkS")
 			(effects
@@
 		(tags "connector JST PH horizontal")
 		(property "Reference" "J3"
-			(at 3 -2.55 0)
+			(at 7.5 -2.55 0)
 			(layer "F.SilkS")
 			(effects
@@
 		)
 		(fp_text user "${REFERENCE}"
-			(at 3 2.5 0)
+			(at 3.5 1.95 0)
 			(layer "F.Fab")
 			(effects
@@
 		(tags "capacitor")
 		(property "Reference" "R3"
-			(at 0 -1.68 0)
+			(at -3 0 0)
 			(layer "F.SilkS")
 			(effects
@@
 		(tags "barrel jack cui dc power")
 		(property "Reference" "J1"
-			(at 0 -2.3 0)
+			(at 7.5 8 0)
 			(layer "F.SilkS")
 			(effects
@@
 		(tags "capacitor")
 		(property "Reference" "R2"
-			(at 0 -1.68 0)
+			(at -3.05 0 0)
 			(layer "F.SilkS")
 			(effects
@@
 		(layer "Edge.Cuts")
 	)
+	(gr_text "SCL"
+		(at 135 54.05 90)
+		(layer "F.SilkS")
+		(effects
+			(font
+				(size 1 1)
+				(thickness 0.15)
+			)
+			(justify left bottom)
+		)
+	)
+	(gr_text "Din"
+		(at 133.5 116 90)
+		(layer "F.SilkS")
+		(effects
+			(font
+				(size 1 1)
+				(thickness 0.15)
+			)
+			(justify left bottom)
+		)
+	)
+	(gr_text "GND"
+		(at 135.5 116 90)
+		(layer "F.SilkS")
+		(effects
+			(font
+				(size 1 1)
+				(thickness 0.15)
+			)
+			(justify left bottom)
+		)
+	)
+	(gr_text "5VDC Out"
+		(at 131.5 116 90)
+		(layer "F.SilkS")
+		(effects
+			(font
+				(size 1 1)
+				(thickness 0.15)
+			)
+			(justify left bottom)
+		)
+	)
+	(gr_text "SDA"
+		(at 133 54.05 90)
+		(layer "F.SilkS")
+		(effects
+			(font
+				(size 1 1)
+				(thickness 0.15)
+			)
+			(justify left bottom)
+		)
+	)
+	(gr_text "GND"
+		(at 108.5 117.5 90)
+		(layer "F.SilkS")
+		(effects
+			(font
+				(size 1 1)
+				(thickness 0.15)
+			)
+			(justify left bottom)
+		)
+	)
+	(gr_text "5VDC In"
+		(at 108.5 110.5 90)
+		(layer "F.SilkS")
+		(effects
+			(font
+				(size 1 1)
+				(thickness 0.15)
+			)
+			(justify left bottom)
+		)
+	)
+	(gr_text "GND"
+		(at 131 54.05 90)
+		(layer "F.SilkS")
+		(effects
+			(font
+				(size 1 1)
+				(thickness 0.15)
+			)
+			(justify left bottom)
+		)
+	)
+	(gr_text "3.3VDC\nOut"
+		(at 138.5 53 90)
+		(layer "F.SilkS")
+		(effects
+			(font
+				(size 1 1)
+				(thickness 0.15)
+			)
+			(justify bottom)
+		)
+	)
+	(gr_text "Yens & Yens"
+		(at 114.5 88.613334 270)
+		(layer "B.SilkS")
+		(effects
+			(font
+				(size 2 2)
+				(thickness 0.4)
+				(bold yes)
+			)
+			(justify left bottom mirror)
+		)
+	)
+	(gr_text "Internship Technical Test Assignment"
+		(at 112 93.613334 270)
+		(layer "B.SilkS")
+		(effects
+			(font
+				(size 1 1)
+				(thickness 0.1)
+			)
+			(justify left bottom mirror)
+		)
+	)
 	(gr_text "pico\nUSB"
 		(at 107 56 0)
@@
 		)
 	)
+	(gr_text "V 1.0"
+		(at 108 83.613334 270)
+		(layer "B.SilkS")
+		(effects
+			(font
+				(size 2 2)
+				(thickness 0.4)
+				(bold yes)
+			)
+			(justify left bottom mirror)
+		)
+	)
 	(gr_text "External\nMPU-6050\nConnection"
 		(at 133.5 65 0)
@@
 		(net 54)
 	)
+	(zone
+		(net 6)
+		(net_name "GNDREF")
+		(layers "F.Cu" "B.Cu")
+		(hatch edge 0.5)
+		(connect_pads
+			(clearance 0.5)
+		)
+		(min_thickness 0.25)
+		(filled_areas_thickness no)
+		(fill yes
+			(thermal_gap 0.5)
+			(thermal_bridge_width 0.5)
+			(island_removal_mode 1)
+			(island_area_min 10)
+		)
+		(polygon
+			(pts
+				(xy 100 50) (xy 140 50) (xy 140 125) (xy 100 125)
+			)
+		)
+	)
 	(embedded_fonts no)

Commit message: Ready for final submition
Other:
- board text added: "(2025-11-27)"
Changed lines of the file:
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@@
 	(title_block
 		(title "Internship Technical Test Assignment")
-		(date "2025-11-26")
-		(rev "1")
+		(date "2025-11-27")
+		(rev "1.0")
 		(company "Yens & Yens")
 	)
@@
 		)
 	)
+	(gr_text "5VDC In"
+		(at 107.2965 110.5 -90)
+		(layer "B.SilkS")
+		(effects
+			(font
+				(size 1 1)
+				(thickness 0.15)
+			)
+			(justify left bottom mirror)
+		)
+	)
+	(gr_text "GND"
+		(at 130.2965 116 -90)
+		(layer "B.SilkS")
+		(effects
+			(font
+				(size 1 1)
+				(thickness 0.15)
+			)
+			(justify left bottom mirror)
+		)
+	)
 	(gr_text "pico\nUSB"
 		(at 107 56 0)
@@
 		)
 	)
+	(gr_text "SDA"
+		(at 133.5 54.05 -90)
+		(layer "B.SilkS")
+		(effects
+			(font
+				(size 1 1)
+				(thickness 0.15)
+			)
+			(justify left bottom mirror)
+		)
+	)
+	(gr_text "GND"
+		(at 135.5 54.05 -90)
+		(layer "B.SilkS")
+		(effects
+			(font
+				(size 1 1)
+				(thickness 0.15)
+			)
+			(justify left bottom mirror)
+		)
+	)
+	(gr_text "(2025-11-27)"
+		(at 106 85 270)
+		(layer "B.SilkS")
+		(effects
+			(font
+				(size 1 1)
+				(thickness 0.1)
+			)
+			(justify left bottom mirror)
+		)
+	)
 	(gr_text "V 1.0"
 		(at 108 83.613334 270)
@@
 		)
 	)
+	(gr_text "3.3VDC\nOut"
+		(at 128 53 -90)
+		(layer "B.SilkS")
+		(effects
+			(font
+				(size 1 1)
+				(thickness 0.15)
+			)
+			(justify bottom mirror)
+		)
+	)
+	(gr_text "5VDC Out"
+		(at 134.2965 116 -90)
+		(layer "B.SilkS")
+		(effects
+			(font
+				(size 1 1)
+				(thickness 0.15)
+			)
+			(justify left bottom mirror)
+		)
+	)
 	(gr_text "External\nMPU-6050\nConnection"
 		(at 133.5 65 0)
@@
 		)
 	)
+	(gr_text "GND"
+		(at 107.2965 117.5 -90)
+		(layer "B.SilkS")
+		(effects
+			(font
+				(size 1 1)
+				(thickness 0.15)
+			)
+			(justify left bottom mirror)
+		)
+	)
+	(gr_text "SCL"
+		(at 131.5 54.05 -90)
+		(layer "B.SilkS")
+		(effects
+			(font
+				(size 1 1)
+				(thickness 0.15)
+			)
+			(justify left bottom mirror)
+		)
+	)
+	(gr_text "Din"
+		(at 132.2965 116 -90)
+		(layer "B.SilkS")
+		(effects
+			(font
+				(size 1 1)
+				(thickness 0.15)
+			)
+			(justify left bottom mirror)
+		)
+	)
